File: pcb/emu-hotswap.sch (KiCad schematic (older format))
At the start: 74 parts, among them J1 TRRS, SW1 SW_Push, SW10 SW_Push, SW11 SW_Push, SW12 SW_Push, SW13 SW_Push, SW14 SW_Push, SW15 SW_Push, SW16 SW_Push, SW17 SW_Push, SW18 SW_Push, SW19 SW_Push, SW2 SW_Push, SW20 SW_Push, SW21 SW_Push, SW22 SW_Push, SW23 SW_Push, SW24 SW_Push, SW25 SW_Push, SW26 SW_Push, SW27 SW_Push, SW28 SW_Push, SW29 SW_Push, SW3 SW_Push, SW30 SW_Push, SW31 SW_Push, SW4 SW_Push, SW5 SW_Push, SW6 SW_Push, SW7 SW_Push, SW8 SW_Push, SW9 SW_Push, U1 ProMicro

Commit message: Work in progress
Parts:
- U1: footprint used_footprints:ProMicro_Dual -> used_footprints:Pro_Micro
Changed lines of the file:
@@
 F 0 "U1" H 1940 2732 60  0000 C CNN
 F 1 "ProMicro" H 1940 2626 60  0000 C CNN
-F 2 "used_footprints:ProMicro_Dual" H 2040 645 60  0001 C CNN
+F 2 "used_footprints:Pro_Micro" H 2040 645 60  0001 C CNN
 F 3 "" H 2040 645 60  0000 C CNN
 	1    1940 1695

Commit message: Roughly cut edges, fixed footprints on the scheme.
Parts:
- added D31: 1N4148, used_footprints:Diode_Hybrid_SOD-123, symbol Device:D_Small
- added SW31: SW_Push, used_footprints:Switch_Mx_Hotswap_1u, symbol Switch:SW_Push
- U1: footprint used_footprints:Pro_Micro -> used_footprints:ArduinoProMicro
- renumbered SW31 to SW32
Connections:
- net labels added: rowF
- wire segments 86 -> 88
- no-connect marks 6 -> 5
Changed lines of the file:
@@
 Text Label 1240 2045 2    50   ~ 0
 rowB
-Text Label 2640 1345 0    50   ~ 0
-rowC
 Text Label 2640 1445 0    50   ~ 0
 rowD
@@
 	1    2830 1245
 	0    1    1    0
-$EndComp
-$Comp
-L Switch:SW_Push SW1
-U 1 1 5DAAE5C1
-P 3745 890
-F 0 "SW1" H 3745 1045 50  0000 C CNN
-F 1 "SW_Push" H 3745 1084 50  0001 C CNN
-F 2 "used_footprints:Switch_Mx_Hotswap_1u" H 3745 1090 50  0001 C CNN
-F 3 "~" H 3745 1090 50  0001 C CNN
-	1    3745 890
-	1    0    0    -1
 $EndComp
 $Comp
@@
 	6945 890  6945 1290
 $Comp
-L Switch:SW_Push SW31
+L Switch:SW_Push SW32
 U 1 1 5DBF73FF
 P 2720 3125
-F 0 "SW31" H 2720 3410 50  0000 C CNN
+F 0 "SW32" H 2720 3410 50  0000 C CNN
 F 1 "SW_Push" H 2720 3319 50  0000 C CNN
 F 2 "used_footprints:Switch_Reset_THT" H 2720 3325 50  0001 C CNN
@@
 Wire Wire Line
 	2830 1245 2640 1245
-NoConn ~ 2640 1645
 NoConn ~ 2640 1745
 NoConn ~ 2640 1845
@@
 F 0 "U1" H 1940 2732 60  0000 C CNN
 F 1 "ProMicro" H 1940 2626 60  0000 C CNN
-F 2 "used_footprints:Pro_Micro" H 2040 645 60  0001 C CNN
+F 2 "used_footprints:ArduinoProMicro" H 2040 645 60  0001 C CNN
 F 3 "" H 2040 645 60  0000 C CNN
 	1    1940 1695
@@
 $EndComp
 NoConn ~ 2640 2045
+Text Label 2640 1345 0    50   ~ 0
+rowC
+$Comp
+L Switch:SW_Push SW31
+U 1 1 603D9F6E
+P 6745 2890
+F 0 "SW31" H 6745 3045 50  0000 C CNN
+F 1 "SW_Push" H 6745 3084 50  0001 C CNN
+F 2 "used_footprints:Switch_Mx_Hotswap_1u" H 6745 3090 50  0001 C CNN
+F 3 "~" H 6745 3090 50  0001 C CNN
+	1    6745 2890
+	1    0    0    -1
+$EndComp
+Connection ~ 6945 2490
+Text Label 3330 3090 0    50   ~ 0
+rowF
+Wire Wire Line
+	6945 2490 6945 2890
+$Comp
+L Device:D_Small D31
+U 1 1 603D9F74
+P 6545 2990
+F 0 "D31" V 6545 2922 50  0000 R CNN
+F 1 "1N4148" V 6500 2922 50  0001 R CNN
+F 2 "used_footprints:Diode_Hybrid_SOD-123" V 6545 2990 50  0001 C CNN
+F 3 "~" V 6545 2990 50  0001 C CNN
+	1    6545 2990
+	0    -1   -1   0
+$EndComp
+Text Label 2640 1645 0    50   ~ 0
+rowF
+Wire Wire Line
+	6545 3090 3330 3090
+$Comp
+L Switch:SW_Push SW1
+U 1 1 5DAAE5C1
+P 3745 890
+F 0 "SW1" H 3745 1045 50  0000 C CNN
+F 1 "SW_Push" H 3745 1084 50  0001 C CNN
+F 2 "used_footprints:Switch_Mx_Hotswap_1u" H 3745 1090 50  0001 C CNN
+F 3 "~" H 3745 1090 50  0001 C CNN
+	1    3745 890
+	1    0    0    -1
+$EndComp
 $EndSCHEMATC

Commit message: Rotated thumb switches to 180 degrees.
Parts:
- D1, D10, D11, D12, D13, D14, D15, D16, D17, D18, D19, D2, D20, D21, D22, D23, D24, D25, D26, D27, D28, D29, D3, D30, D31, D4, D5, D6, D7, D8, D9: footprint used_footprints:Diode_Hybrid_SOD-123 -> used_footprints:D3_TH_SMD
- SW1, SW11, SW12, SW13, SW14, SW16, SW17, SW18, SW19, SW2, SW20, SW21, SW22, SW23, SW24, SW25, SW26, SW27, SW28, SW29, SW3, SW30, SW31, SW4, SW5, SW6, SW7, SW8, SW9: footprint used_footprints:Switch_Mx_Hotswap_1u -> used_footprints:CherryMX_MidHeight_Hotswap_1u
- SW10, SW15: footprint used_footprints:Switch_Mx_Hotswap_1u -> used_footprints:CherryMX_MidHeight_Hotswap_1.25u

Commit message: Routing...
Parts:
- added HM6: CaseHole, used_footprints:Hole_Mount_M4, symbol Mechanical:MountingHole
Changed lines of the file:
@@
+	1    0    0    -1
+$EndComp
+$Comp
+L Mechanical:MountingHole HM6
+U 1 1 60492C63
+P 7370 1840
+F 0 "HM6" H 7470 1886 50  0000 L CNN
+F 1 "CaseHole" H 7470 1795 50  0000 L CNN
+F 2 "used_footprints:Hole_Mount_M4" H 7370 1840 50  0001 C CNN
+F 3 "~" H 7370 1840 50  0001 C CNN
+	1    7370 1840
 	1    0    0    -1
 $EndComp

Commit message: Routing dual ProMicro footprint
Parts:
- U1: footprint used_footprints:ArduinoProMicro -> used_footprints:ArduinoProMicro_dual
Changed lines of the file:
@@
 F 0 "U1" H 1940 2732 60  0000 C CNN
 F 1 "ProMicro" H 1940 2626 60  0000 C CNN
-F 2 "used_footprints:ArduinoProMicro" H 2040 645 60  0001 C CNN
+F 2 "used_footprints:ArduinoProMicro_dual" H 2040 645 60  0001 C CNN
 F 3 "" H 2040 645 60  0000 C CNN
 	1    1940 1695

Commit message: Started new simple and weird design.
Parts:
- U1: footprint used_footprints:ArduinoProMicro_dual -> used_footprints:ProMicro_Dual
Changed lines of the file:
@@
 F 0 "U1" H 1940 2732 60  0000 C CNN
 F 1 "ProMicro" H 1940 2626 60  0000 C CNN
-F 2 "used_footprints:ArduinoProMicro_dual" H 2040 645 60  0001 C CNN
+F 2 "used_footprints:ProMicro_Dual" H 2040 645 60  0001 C CNN
 F 3 "" H 2040 645 60  0000 C CNN
 	1    1940 1695

Commit message: Holes.
Parts:
- added HM10, HM11, HM12, HM7, HM8, HM9: CaseHole, used_footprints:Hole_Mount_M4, symbol Mechanical:MountingHole
Changed lines of the file:
@@
+	1    0    0    -1
+$EndComp
+$Comp
+L Mechanical:MountingHole HM7
+U 1 1 60415820
+P 8215 1190
+F 0 "HM7" H 8315 1236 50  0000 L CNN
+F 1 "CaseHole" H 8315 1145 50  0000 L CNN
+F 2 "used_footprints:Hole_Mount_M4" H 8215 1190 50  0001 C CNN
+F 3 "~" H 8215 1190 50  0001 C CNN
+	1    8215 1190
+	1    0    0    -1
+$EndComp
+$Comp
+L Mechanical:MountingHole HM8
+U 1 1 60415826
+P 8215 1380
+F 0 "HM8" H 8315 1426 50  0000 L CNN
+F 1 "CaseHole" H 8315 1335 50  0000 L CNN
+F 2 "used_footprints:Hole_Mount_M4" H 8215 1380 50  0001 C CNN
+F 3 "~" H 8215 1380 50  0001 C CNN
+	1    8215 1380
+	1    0    0    -1
+$EndComp
+$Comp
+L Mechanical:MountingHole HM9
+U 1 1 6041582C
+P 8215 1580
+F 0 "HM9" H 8315 1626 50  0000 L CNN
+F 1 "CaseHole" H 8315 1535 50  0000 L CNN
+F 2 "used_footprints:Hole_Mount_M4" H 8215 1580 50  0001 C CNN
+F 3 "~" H 8215 1580 50  0001 C CNN
+	1    8215 1580
+	1    0    0    -1
+$EndComp
+$Comp
+L Mechanical:MountingHole HM10
+U 1 1 60415832
+P 8215 1785
+F 0 "HM10" H 8315 1831 50  0000 L CNN
+F 1 "CaseHole" H 8315 1740 50  0000 L CNN
+F 2 "used_footprints:Hole_Mount_M4" H 8215 1785 50  0001 C CNN
+F 3 "~" H 8215 1785 50  0001 C CNN
+	1    8215 1785
+	1    0    0    -1
+$EndComp
+$Comp
+L Mechanical:MountingHole HM11
+U 1 1 60415838
+P 8215 1975
+F 0 "HM11" H 8315 2021 50  0000 L CNN
+F 1 "CaseHole" H 8315 1930 50  0000 L CNN
+F 2 "used_footprints:Hole_Mount_M4" H 8215 1975 50  0001 C CNN
+F 3 "~" H 8215 1975 50  0001 C CNN
+	1    8215 1975
+	1    0    0    -1
+$EndComp
+$Comp
+L Mechanical:MountingHole HM12
+U 1 1 6041583E
+P 8220 2170
+F 0 "HM12" H 8320 2216 50  0000 L CNN
+F 1 "CaseHole" H 8320 2125 50  0000 L CNN
+F 2 "used_footprints:Hole_Mount_M4" H 8220 2170 50  0001 C CNN
+F 3 "~" H 8220 2170 50  0001 C CNN
+	1    8220 2170
 	1    0    0    -1
 $EndComp
