File: cover/cover/cover.kicad_pcb (KiCad board)
At the start: 2 copper layers, 52.7 x 95.2 mm, 5 parts

Commit message: Multiple fixes...
Parts:
- removed H13, H16: MountingHole, used_footprints:M2_HOLE_PCB
- removed HM3: CaseHole, used_footprints:M2_HOLE_PCB
- moved H15 4.86 mm to (246.7, 97.2)
- moved HM12 4.25 mm to (228.0, 74.8)
Other:
- board size 52.7 x 95.2 mm -> 35.4 x 51.7 mm
Changed lines of the file:
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@@
   (general
     (thickness 1.6)
-    (drawings 26)
+    (drawings 15)
     (tracks 0)
     (zones 0)
-    (modules 5)
+    (modules 2)
     (nets 1)
   )
@@
   )
   (module used_footprints:M2_HOLE_PCB (layer F.Cu)
-    (at 230.15 74.8)
-    (fp_text reference H16 (at 0 2.7) (layer F.SilkS) hide
+    (at 246.7 97.25 9)
+    (fp_text reference H15 (at 0 2.7 9) (layer F.SilkS) hide
       (effects (font (size 1 1) (thickness 0.15)))
     )
-    (fp_text value MountingHole (at 0 -2.6) (layer F.Fab) hide
+    (fp_text value MountingHole (at 0 -2.6 9) (layer F.Fab) hide
       (effects (font (size 1 1) (thickness 0.15)))
     )
-    (pad "" thru_hole circle (at 0 0) (size 4 4) (drill 2.2) (layers *.Cu *.Mask))
+    (pad "" thru_hole circle (at 0.033741 0.106591 9) (size 4 4) (drill 2.2) (layers *.Cu *.Mask))
   )
   (module used_footprints:M2_HOLE_PCB (layer F.Cu)
-    (at 243.895 105.37)
-    (fp_text reference HM3 (at 0 2.7) (layer F.SilkS) hide
-      (effects (font (size 1 1) (thickness 0.15)))
-    )
-    (fp_text value CaseHole (at 0 -2.6) (layer F.Fab) hide
-      (effects (font (size 1 1) (thickness 0.15)))
-    )
-    (pad "" thru_hole circle (at 0 0) (size 4 4) (drill 2.2) (layers *.Cu *.Mask))
-  )
-  (module used_footprints:M2_HOLE_PCB (layer F.Cu)
-    (at 223.75 74.8)
+    (at 228 74.8)
     (fp_text reference HM12 (at 0 2.7) (layer F.SilkS) hide
       (effects (font (size 1 1) (thickness 0.15)))
@@
     (pad "" thru_hole circle (at 0 0) (size 4 4) (drill 2.2) (layers *.Cu *.Mask))
   )
-  (module used_footprints:M2_HOLE_PCB (layer F.Cu)
-    (at 251.35 95.85 9)
-    (fp_text reference H15 (at 0 2.7 9) (layer F.SilkS) hide
-      (effects (font (size 1 1) (thickness 0.15)))
-    )
-    (fp_text value MountingHole (at 0 -2.6 9) (layer F.Fab) hide
-      (effects (font (size 1 1) (thickness 0.15)))
-    )
-    (pad "" thru_hole circle (at 0 0 9) (size 4 4) (drill 2.2) (layers *.Cu *.Mask))
-  )
-  (module used_footprints:M2_HOLE_PCB (layer F.Cu)
-    (at 233.95 98.65 36)
-    (fp_text reference H13 (at 0 2.7 36) (layer F.SilkS) hide
-      (effects (font (size 1 1) (thickness 0.15)))
-    )
-    (fp_text value MountingHole (at 0 -2.6 36) (layer F.Fab) hide
-      (effects (font (size 1 1) (thickness 0.15)))
-    )
-    (pad "" thru_hole circle (at 0 0 36) (size 4 4) (drill 2.2) (layers *.Cu *.Mask))
-  )
-  (gr_line (start 254.95 95.05) (end 251.9 104.3) (layer Edge.Cuts) (width 0.05))
+  (gr_line (start 250.610456 104.28905) (end 251.52 104.75) (layer Edge.Cuts) (width 0.05))
+  (gr_line (start 219.730203 57.134768) (end 219.59 56.25) (layer Edge.Cuts) (width 0.05))
+  (gr_line (start 252.2 103.42) (end 251.52 104.75) (layer Edge.Cuts) (width 0.05))
+  (gr_line (start 227.4 56.25) (end 219.59 56.25) (layer Edge.Cuts) (width 0.05))
+  (gr_arc (start 247.990448 55.013936) (end 249.965825 54.701067) (angle -90) (layer Edge.Cuts) (width 0.05))
+  (gr_line (start 232.832337 84.363517) (end 223.57 81.35) (layer Edge.Cuts) (width 0.05))
+  (gr_arc (start 248.335778 101.268003) (end 252.2 103.42) (angle -15.75657092) (layer Edge.Cuts) (width 0.05))
+  (gr_line (start 254.95 87.7) (end 252.639175 102.289804) (layer Edge.Cuts) (width 0.05))
+  (gr_line (start 235.38 96.53) (end 250.610456 104.28905) (layer Edge.Cuts) (width 0.05))
+  (gr_line (start 247.677579 53.038559) (end 227.4 56.25) (layer Edge.Cuts) (width 0.05))
+  (gr_line (start 233.59 85.21) (end 235.38 96.53) (layer Edge.Cuts) (width 0.05))
   (gr_line (start 249.965825 54.701067) (end 254.95 86.2) (layer Edge.Cuts) (width 0.05))
-  (gr_line (start 247.677579 53.038559) (end 227.4 56.25) (layer Edge.Cuts) (width 0.05))
-  (gr_line (start 202.25 56.249998) (end 209.65 56.25) (layer Edge.Cuts) (width 0.05))
-  (gr_line (start 234.283043 134.070973) (end 223.996802 148.22877) (layer Edge.Cuts) (width 0.05))
-  (gr_line (start 242.7 122.45) (end 234.283043 134.070973) (layer Edge.Cuts) (width 0.05))
-  (gr_line (start 254.95 86.2) (end 254.95 95.05) (layer Edge.Cuts) (width 0.05))
-  (gr_arc (start 247.990448 55.013936) (end 249.965825 54.701067) (angle -90) (layer Edge.Cuts) (width 0.05))
-  (gr_line (start 251.9 104.3) (end 242.7 122.45) (layer Edge.Cuts) (width 0.05))
-  (gr_line (start 227.4 56.25) (end 209.65 56.25) (layer Edge.Cuts) (width 0.05))
-  (gr_arc (start 233.074311 134.022948) (end 233.883328 134.610732) (angle -22.89982715) (layer Edge.Cuts) (width 0.05))
-  (gr_line (start 234.05 133.8) (end 234.025367 133.713932) (layer Edge.Cuts) (width 0.05))
-  (gr_arc (start 233.074311 134.022948) (end 234.025367 133.713932) (angle -36.00009061) (layer Edge.Cuts) (width 0.05))
-  (gr_line (start 232.685901 107.932607) (end 227.34 105.21) (layer Edge.Cuts) (width 0.05))
-  (gr_line (start 233.662096 133.21393) (end 224.24 126.36) (layer Edge.Cuts) (width 0.05))
-  (gr_line (start 202.25 56.249998) (end 208.71 56.25) (layer Edge.Cuts) (width 0.05))
-  (gr_line (start 209.65 77.26) (end 216.690846 79.552671) (layer Edge.Cuts) (width 0.05))
-  (gr_arc (start 232.231911 108.823614) (end 233.122916 109.277604) (angle -90) (layer Edge.Cuts) (width 0.05))
-  (gr_line (start 232.906359 84.821411) (end 216.690846 79.552671) (layer Edge.Cuts) (width 0.05))
-  (gr_line (start 227.34 105.21) (end 233.548399 86.081484) (layer Edge.Cuts) (width 0.05))
-  (gr_line (start 223.996802 148.22877) (end 233.883328 134.610732) (layer Edge.Cuts) (width 0.05))
-  (gr_arc (start 232.597343 85.772468) (end 233.548399 86.081484) (angle -90) (layer Edge.Cuts) (width 0.05))
-  (gr_arc (start 208.65 57.25) (end 209.65 57.31) (angle -90) (layer Edge.Cuts) (width 0.05))
-  (gr_line (start 209.65 57.31) (end 209.65 77.26) (layer Edge.Cuts) (width 0.05))
-  (gr_line (start 224.24 126.36) (end 233.122916 109.277604) (layer Edge.Cuts) (width 0.05))
-  (gr_line (start 234.05 134.25) (end 234.05 133.8) (layer Edge.Cuts) (width 0.05))
+  (gr_line (start 254.95 86.2) (end 254.95 87.7) (layer Edge.Cuts) (width 0.05))
+  (gr_arc (start 232.571527 85.359283) (end 233.59 85.21) (angle -67) (layer Edge.Cuts) (width 0.05))
+  (gr_line (start 219.730203 57.134768) (end 223.57 81.35) (layer Edge.Cuts) (width 0.05))
 )
